Commit message: finished

File: data/robot/body.urdf (robot description, URDF)
Before this commit: robot robot, 3 links, 2 joints
Links:
- added link backleglower, mass 1; collision box size=0.2 0.2 1; visual box size=0.2 0.2 1
- added link frontleglower, mass 1; collision box size=0.2 0.2 1; visual box size=0.2 0.2 1
- added link leftleg, mass 1; collision box size=1 0.2 0.2; visual box size=1 0.2 0.2
- added link leftleglower, mass 1; collision box size=0.2 0.2 1; visual box size=0.2 0.2 1
- added link rightleg, mass 1; collision box size=1 0.2 0.2; visual box size=1 0.2 0.2
- added link rightleglower, mass 1; collision box size=0.2 0.2 1; visual box size=0.2 0.2 1
- link backleg: geometry collision box size=0.2 1 0.2; visual box size=0.2 1 0.2
- link frontleg: geometry collision box size=0.2 1 0.2; visual box size=0.2 1 0.2
Joints:
- added joint backleg_backleglower: type revolute, parent backleg, child backleglower, origin xyz=0 -1 0 rpy=0 0 0, axis 0 1 0, limit lower=-3.14159 upper=3.14159 effort=0.0 velocity=0.0
- added joint frontleg_frontleglower: type revolute, parent frontleg, child frontleglower, origin xyz=0 1 0 rpy=0 0 0, axis 0 1 0, limit lower=-3.14159 upper=3.14159 effort=0.0 velocity=0.0
- added joint leftleg_leftleglower: type revolute, parent leftleg, child leftleglower, origin xyz=-1 0 0 rpy=0 0 0, axis 0 1 0, limit lower=-3.14159 upper=3.14159 effort=0.0 velocity=0.0
- added joint rightleg_rightleglower: type revolute, parent rightleg, child rightleglower, origin xyz=1 0 0 rpy=0 0 0, axis 0 1 0, limit lower=-3.14159 upper=3.14159 effort=0.0 velocity=0.0
- added joint torso_leftleg: type revolute, parent torso, child leftleg, origin xyz=-0.5 0 1 rpy=0 0 0, axis 0 1 0, limit lower=-3.14159 upper=3.14159 effort=0.0 velocity=0.0
- added joint torso_rightleg: type revolute, parent torso, child rightleg, origin xyz=0.5 0 1 rpy=0 0 0, axis 0 1 0, limit lower=-3.14159 upper=3.14159 effort=0.0 velocity=0.0
- joint torso_backleg: axis 0 1 0 -> 1 0 0; origin xyz=0.5 0 1 rpy=0 0 0 -> xyz=0 -0.5 1 rpy=0 0 0
- joint torso_frontleg: axis 0 1 0 -> 1 0 0; origin xyz=-0.5 0 1 rpy=0 0 0 -> xyz=0 0.5 1 rpy=0 0 0
