Commit message: simulate 3 box robot

File: body.urdf (robot description, URDF)
Before this commit: robot robot, 7 links, 6 joints
Links:
- removed link link0
- removed link link1
- removed link link2
- removed link link3
- removed link link4
- removed link link5
- removed link link6
- added link backleg, mass 1; collision box size=1 1 1; visual box size=1 1 1
- added link frontleg, mass 1; collision box size=1 1 1; visual box size=1 1 1
- added link torso, mass 1; collision box size=1 1 1; visual box size=1 1 1
Joints:
- removed joint link0_link1
- removed joint link1_link2
- removed joint link2_link3
- removed joint link3_link4
- removed joint link4_link5
- removed joint link5_link6
- added joint torso_backleg: type revolute, parent torso, child backleg, origin xyz=0 0.5 1 rpy=0 0 0, axis 0 1 0, limit lower=-3.14159 upper=3.14159 effort=0.0 velocity=0.0
- added joint torso_frontleg: type revolute, parent torso, child frontleg, origin xyz=0 -0.5 1 rpy=0 0 0, axis 0 1 0, limit lower=-3.14159 upper=3.14159 effort=0.0 velocity=0.0

Commit message: add backleg sensor

File: body.urdf (robot description, URDF)
Before this commit: robot robot, 3 links, 2 joints
Joints:
- joint torso_backleg: axis 1 0 0 -> 0 1 0; origin xyz=0 0.5 1 rpy=0 0 0 -> xyz=0.5 0 1 rpy=0 0 0
- joint torso_frontleg: axis 1 0 0 -> 0 1 0; origin xyz=0 -0.5 1 rpy=0 0 0 -> xyz=-0.5 0 1 rpy=0 0 0

Commit message: working genetic algorithm

File: body.urdf (robot description, URDF)
Before this commit: robot robot, 25 links, 24 joints
Links:
- removed link backleftcoxa
- removed link backleftfemur
- removed link backlefttibia
- removed link backrightcoxa
- removed link backrightfemur
- removed link backrighttibia
- removed link frontleftcoxa
- removed link frontleftfemur
- removed link frontlefttibia
- removed link frontrightcoxa
- removed link frontrightfemur
- removed link frontrighttibia
- removed link leftbacktibia
- removed link leftfronttibia
- removed link rightbacktibia
- removed link rightfronttibia
- link leftbackfemur: geometry collision box size=2 0.2 0.2; visual box size=2 0.2 0.2
- link leftfrontfemur: geometry collision box size=2 0.2 0.2; visual box size=2 0.2 0.2
- link rightbackfemur: geometry collision box size=2 0.2 0.2; visual box size=2 0.2 0.2
- link rightfrontfemur: geometry collision box size=2 0.2 0.2; visual box size=2 0.2 0.2
- link torso: geometry collision box size=1 1 0.5; visual box size=1 1 0.5
Joints:
- removed joint backleftcoxa_backleftfemur
- removed joint backleftfemur_backlefttibia
- removed joint backrightcoxa_backrightfemur
- removed joint backrightfemur_backrighttibia
- removed joint frontleftcoxa_frontleftfemur
- removed joint frontleftfemur_frontlefttibia
- removed joint frontrightcoxa_frontrightfemur
- removed joint frontrightfemur_frontrighttibia
- removed joint leftbackfemur_leftbacktibia
- removed joint leftfrontfemur_leftfronttibia
- removed joint rightbackfemur_rightbacktibia
- removed joint rightfrontfemur_rightfronttibia
- removed joint torso_backleftcoxa
- removed joint torso_backrightcoxa
- removed joint torso_frontleftcoxa
- removed joint torso_frontrightcoxa
- joint torso_leftbackcoxa: origin xyz=-0.5 -0.3 1 rpy=0 0 0 -> xyz=-0.5 -0.4 1 rpy=0 0 0
- joint torso_leftfrontcoxa: origin xyz=-0.5 0.3 1 rpy=0 0 0 -> xyz=-0.5 0.4 1 rpy=0 0 0
- joint torso_rightbackcoxa: origin xyz=0.5 -0.3 1 rpy=0 0 0 -> xyz=0.5 -0.4 1 rpy=0 0 0
- joint torso_rightfrontcoxa: origin xyz=0.5 0.3 1 rpy=0 0 0 -> xyz=0.5 0.4 1 rpy=0 0 0
